File: Hardware/Production/esp32_lora_gateway-Panel.brd (EAGLE design)
At the start: 90.9 x 120.5 mm, 486 parts, among them J15 U.FL, J21 U.FL, J27 U.FL, J33 U.FL, J5 U.FL, J7 U.FL, Q1 MBT3904DW1T1, Q2 MBT3904DW1T1, Q3 MBT3904DW1T1, Q4 MBT3904DW1T1, Q5 MBT3904DW1T1, Q6 MBT3904DW1T1, U1 ESP-WROOM-32NARROW, U10 RFM96W, U11 3.3V, U12 CH340C, U13 ESP-WROOM-32NARROW, U14 RFM96W, U15 3.3V, U16 CH340C, U17 ESP-WROOM-32NARROW, U18 RFM96W, U19 3.3V, U2 RFM96W, U20 CH340C, U21 ESP-WROOM-32NARROW, U22 RFM96W, U23 3.3V, U24 CH340C, U3 3.3V, U4 ESP-WROOM-32NARROW, U5 CH340C, U6 RFM96W, U7 3.3V, U8 CH340C, U9 ESP-WROOM-32NARROW

Commit message: Changing blue LED to green.
Parts:
- D11, D2, D3, D5, D7, D9: value BLUE -> GREEN
Changed lines of the file:
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@@
 <?xml version="1.0" encoding="utf-8"?>
 <!DOCTYPE eagle SYSTEM "eagle.dtd">
-<eagle version="9.0.1">
+<eagle version="9.1.1">
 <drawing>
 <settings>
@@
 <param name="checkStop" value="0"/>
 <param name="checkValues" value="0"/>
+<param name="checkNames" value="1"/>
+<param name="checkWireStubs" value="1"/>
+<param name="checkPolygonWidth" value="0"/>
 <param name="useDiameter" value="13"/>
 <param name="maxErrors" value="50"/>
@@
 <attribute name="PROD_ID" value="SWCH-13065" x="1.905" y="3.175" size="1.778" layer="27" font="vector" ratio="15" rot="R270" display="off"/>
 </element>
-<element name="D3" library="SparkFun-LED" package="LED-0603" value="BLUE" x="19.304" y="2.54" rot="R90">
-<attribute name="PROD_ID" value="DIO-08575" x="19.304" y="0" size="1.778" layer="27" font="vector" ratio="15" rot="R90" display="off"/>
+<element name="D3" library="SparkFun-LED" package="LED-0603" value="GREEN" x="19.304" y="2.54" rot="R90">
+<attribute name="PROD_ID" value="DIO-00821" x="19.304" y="0" size="1.778" layer="27" font="vector" ratio="15" rot="R90" display="off"/>
 </element>
 <element name="R4" library="SparkFun-Resistors" package="0603" value="1k" x="17.78" y="2.54" rot="R270">
@@
 <attribute name="PROD_ID" value="SWCH-13065" x="27.793009375" y="3.175" size="1.778" layer="27" font="vector" ratio="15" rot="R270" display="off"/>
 </element>
-<element name="D2" library="SparkFun-LED" package="LED-0603" value="BLUE" x="45.192009375" y="2.54" rot="R90">
-<attribute name="PROD_ID" value="DIO-08575" x="45.192009375" y="0" size="1.778" layer="27" font="vector" ratio="15" rot="R90" display="off"/>
+<element name="D2" library="SparkFun-LED" package="LED-0603" value="GREEN" x="45.192009375" y="2.54" rot="R90">
+<attribute name="PROD_ID" value="DIO-00821" x="45.192009375" y="0" size="1.778" layer="27" font="vector" ratio="15" rot="R90" display="off"/>
 </element>
 <element name="R9" library="SparkFun-Resistors" package="0603" value="1k" x="43.668009375" y="2.54" rot="R270">
@@
 <attribute name="PROD_ID" value="SWCH-13065" x="53.68099375" y="3.175" size="1.778" layer="27" font="vector" ratio="15" rot="R270" display="off"/>
 </element>
-<element name="D5" library="SparkFun-LED" package="LED-0603" value="BLUE" x="71.07999375" y="2.54" rot="R90">
-<attribute name="PROD_ID" value="DIO-08575" x="71.07999375" y="0" size="1.778" layer="27" font="vector" ratio="15" rot="R90" display="off"/>
+<element name="D5" library="SparkFun-LED" package="LED-0603" value="GREEN" x="71.07999375" y="2.54" rot="R90">
+<attribute name="PROD_ID" value="DIO-00821" x="71.07999375" y="0" size="1.778" layer="27" font="vector" ratio="15" rot="R90" display="off"/>
 </element>
 <element name="R16" library="SparkFun-Resistors" package="0603" value="1k" x="69.55599375" y="2.54" rot="R270">
@@
 <attribute name="PROD_ID" value="SWCH-13065" x="1.905" y="52.375003125" size="1.778" layer="27" font="vector" ratio="15" rot="R270" display="off"/>
 </element>
-<element name="D7" library="SparkFun-LED" package="LED-0603" value="BLUE" x="19.304" y="51.740003125" rot="R90">
-<attribute name="PROD_ID" value="DIO-08575" x="19.304" y="49.200003125" size="1.778" layer="27" font="vector" ratio="15" rot="R90" display="off"/>
+<element name="D7" library="SparkFun-LED" package="LED-0603" value="GREEN" x="19.304" y="51.740003125" rot="R90">
+<attribute name="PROD_ID" value="DIO-00821" x="19.304" y="49.200003125" size="1.778" layer="27" font="vector" ratio="15" rot="R90" display="off"/>
 </element>
 <element name="R25" library="SparkFun-Resistors" package="0603" value="1k" x="17.78" y="51.740003125" rot="R270">
@@
 <attribute name="PROD_ID" value="SWCH-13065" x="27.793009375" y="52.375003125" size="1.778" layer="27" font="vector" ratio="15" rot="R270" display="off"/>
 </element>
-<element name="D9" library="SparkFun-LED" package="LED-0603" value="BLUE" x="45.192009375" y="51.740003125" rot="R90">
-<attribute name="PROD_ID" value="DIO-08575" x="45.192009375" y="49.200003125" size="1.778" layer="27" font="vector" ratio="15" rot="R90" display="off"/>
+<element name="D9" library="SparkFun-LED" package="LED-0603" value="GREEN" x="45.192009375" y="51.740003125" rot="R90">
+<attribute name="PROD_ID" value="DIO-00821" x="45.192009375" y="49.200003125" size="1.778" layer="27" font="vector" ratio="15" rot="R90" display="off"/>
 </element>
 <element name="R32" library="SparkFun-Resistors" package="0603" value="1k" x="43.668009375" y="51.740003125" rot="R270">
@@
 <attribute name="PROD_ID" value="SWCH-13065" x="53.68099375" y="52.375003125" size="1.778" layer="27" font="vector" ratio="15" rot="R270" display="off"/>
 </element>
-<element name="D11" library="SparkFun-LED" package="LED-0603" value="BLUE" x="71.07999375" y="51.740003125" rot="R90">
-<attribute name="PROD_ID" value="DIO-08575" x="71.07999375" y="49.200003125" size="1.778" layer="27" font="vector" ratio="15" rot="R90" display="off"/>
+<element name="D11" library="SparkFun-LED" package="LED-0603" value="GREEN" x="71.07999375" y="51.740003125" rot="R90">
+<attribute name="PROD_ID" value="DIO-00821" x="71.07999375" y="49.200003125" size="1.778" layer="27" font="vector" ratio="15" rot="R90" display="off"/>
 </element>
 <element name="R39" library="SparkFun-Resistors" package="0603" value="1k" x="69.55599375" y="51.740003125" rot="R270">
@@
 </signal>
 </signals>
+<mfgpreviewcolors>
+<mfgpreviewcolor name="soldermaskcolor" color="0xC8008000"/>
+<mfgpreviewcolor name="silkscreencolor" color="0xFFFEFEFE"/>
+<mfgpreviewcolor name="backgroundcolor" color="0xFF282828"/>
+<mfgpreviewcolor name="coppercolor" color="0xFFFFBF00"/>
+<mfgpreviewcolor name="substratecolor" color="0xFF786E46"/>
+</mfgpreviewcolors>
 </board>
 </drawing>
