File: Hardware/esp32_lora_gateway.brd (EAGLE design)
At the start: 25.4 x 46.2 mm, 81 parts, among them J5 U.FL, Q2 MBT3904DW1T1, U1 ESP-WROOM-32NARROW, U2 RFM96W, U3 3.3V, U5 CH340C

Commit message: Changing blue LED to green.
Parts:
- D3: value BLUE -> GREEN
Changed lines of the file:
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@@
 <?xml version="1.0" encoding="utf-8"?>
 <!DOCTYPE eagle SYSTEM "eagle.dtd">
-<eagle version="9.0.1">
+<eagle version="9.1.1">
 <drawing>
 <settings>
@@
 <param name="checkStop" value="0"/>
 <param name="checkValues" value="0"/>
+<param name="checkNames" value="1"/>
+<param name="checkWireStubs" value="1"/>
+<param name="checkPolygonWidth" value="0"/>
 <param name="useDiameter" value="13"/>
 <param name="maxErrors" value="50"/>
@@
 <attribute name="PROD_ID" value="SWCH-13065" x="1.905" y="3.175" size="1.778" layer="27" font="vector" ratio="15" rot="R270" display="off"/>
 </element>
-<element name="D3" library="SparkFun-LED" package="LED-0603" value="BLUE" x="19.304" y="2.54" rot="R90">
-<attribute name="PROD_ID" value="DIO-08575" x="19.304" y="0" size="1.778" layer="27" font="vector" ratio="15" rot="R90" display="off"/>
+<element name="D3" library="SparkFun-LED" package="LED-0603" value="GREEN" x="19.304" y="2.54" rot="R90">
+<attribute name="PROD_ID" value="DIO-00821" x="19.304" y="0" size="1.778" layer="27" font="vector" ratio="15" rot="R90" display="off"/>
 </element>
 <element name="R4" library="SparkFun-Resistors" package="0603" value="1k" x="17.78" y="2.54" rot="R270">
@@
 </signal>
 </signals>
+<mfgpreviewcolors>
+<mfgpreviewcolor name="soldermaskcolor" color="0xC8008000"/>
+<mfgpreviewcolor name="silkscreencolor" color="0xFFFEFEFE"/>
+<mfgpreviewcolor name="backgroundcolor" color="0xFF282828"/>
+<mfgpreviewcolor name="coppercolor" color="0xFFFFBF00"/>
+<mfgpreviewcolor name="substratecolor" color="0xFF786E46"/>
+</mfgpreviewcolors>
 </board>
 </drawing>

Commit message: Moving part value text for assembly sheet. Set sch version.
Parts:
- J1: value (none) -> USB
- J3: value (none) -> QWIIC
- S2: value RESET -> 0
